Commit message: Publish wrist RGB-D grasping workspace with SAM and local color workflows

File: src/X5A/urdf/X5A_moveit.urdf (robot description, URDF)
Before this commit: robot X5A, 10 links, 9 joints
Links:
- link link6: mass 0.44089 -> 0.66589

File: src/X5A/urdf/X5A_moveit.urdf.xacro (robot description, xacro)
@@ -341,6 +341,9 @@
         xyz="0.041697 2.4368E-05 0.00014464"
         rpy="0 0 0" />
-      <mass
-        value="0.44089" />
+      <!-- Gemini 345LG mounted on link6: add approximately 0.225 kg.
+           Mass-only approximation; COM and inertia retain the original values
+           until the camera mounting offset and inertia are measured. -->
+      <mass
+        value="0.66589" />
       <inertia
         ixx="0.00038"

File: src/x5a_moveit_config/config/X5A.urdf.xacro (robot description, xacro)
@@ -342,6 +342,9 @@
         xyz="0.041697 2.4368E-05 0.00014464"
         rpy="0 0 0" />
-      <mass
-        value="0.44089" />
+      <!-- Gemini 345LG mounted on link6: add approximately 0.225 kg.
+           Mass-only approximation; COM and inertia retain the original values
+           until the camera mounting offset and inertia are measured. -->
+      <mass
+        value="0.66589" />
       <inertia
         ixx="0.00038"
